File: HC-06_Arduino_UNO_Adapter.brd (EAGLE design)
At the start: 52.6 x 23.4 mm, 14 parts

Commit message: minor changes
Routing:
- net GND: track 79.8 -> 79.2 mm
Other:
- board size 52.6 x 23.4 mm -> 52.8 x 23.4 mm
Changed lines of the file:
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@@
 <text x="46.101" y="15.367" size="1.016" layer="25">GND</text>
 <text x="46.101" y="17.907" size="1.016" layer="25">GND</text>
-<wire x1="0.127" y1="1.397" x2="1.651" y2="0.127" width="0" layer="20" curve="90"/>
-<wire x1="1.651" y1="0.127" x2="51.435" y2="0.127" width="0" layer="20"/>
-<wire x1="51.435" y1="0.127" x2="52.705" y2="0.889" width="0" layer="20" curve="90"/>
-<wire x1="52.705" y1="0.889" x2="52.705" y2="19.939" width="0" layer="20"/>
-<wire x1="49.149" y1="23.495" x2="12.827" y2="23.495" width="0" layer="20"/>
-<wire x1="12.827" y1="23.495" x2="11.303" y2="22.225" width="0" layer="20" curve="90"/>
-<wire x1="11.303" y1="22.225" x2="7.874" y2="19.177" width="0" layer="20" curve="-90"/>
-<wire x1="7.874" y1="19.177" x2="1.905" y2="19.177" width="0" layer="20"/>
-<wire x1="1.905" y1="19.177" x2="0.127" y2="17.907" width="0" layer="20" curve="90"/>
-<wire x1="0.127" y1="17.907" x2="0.127" y2="1.397" width="0" layer="20"/>
 <text x="10.795" y="18.923" size="0.8636" layer="25">BT_TX</text>
 <text x="10.795" y="12.065" size="0.8636" layer="25">BT_RX</text>
@@
 HC-05/HC-06 Bluetooth module
 Arduino UNO adapter</text>
-<wire x1="52.705" y1="19.939" x2="49.149" y2="23.495" width="0" layer="20"/>
 <text x="30.353" y="7.747" size="1.27" layer="25" rot="R90">HC-05/06</text>
 <text x="45.847" y="21.463" size="1.27" layer="125" ratio="10">KEY</text>
@@
 <text x="44.6786" y="10.0584" size="0.8128" layer="125" ratio="10" rot="R90">R6</text>
 <text x="38.481" y="21.209" size="1.27" layer="125" ratio="10">S1</text>
+<wire x1="1.524" y1="0" x2="0" y2="1.524" width="0.254" layer="20" curve="-90"/>
+<wire x1="0" y1="1.524" x2="0" y2="17.018" width="0.254" layer="20"/>
+<wire x1="0" y1="17.018" x2="6.35" y2="23.368" width="0.254" layer="20" curve="-90"/>
+<wire x1="6.35" y1="23.368" x2="48.768" y2="23.368" width="0.254" layer="20"/>
+<wire x1="48.768" y1="23.368" x2="52.832" y2="19.304" width="0.254" layer="20" curve="-90"/>
+<wire x1="52.832" y1="19.304" x2="52.832" y2="6.858" width="0.254" layer="20"/>
+<wire x1="52.832" y1="6.858" x2="45.974" y2="0" width="0.254" layer="20" curve="-90"/>
+<wire x1="45.974" y1="0" x2="1.524" y2="0" width="0.254" layer="20"/>
 </plain>
 <attributes>
@@
 <contactref element="HC-06" pad="22"/>
 <wire x1="20.701" y1="4.225" x2="21.59" y2="4.225" width="0.8128" layer="1"/>
-<wire x1="21.59" y1="4.225" x2="23.749" y2="5.715" width="0.8128" layer="1"/>
-<wire x1="23.749" y1="5.715" x2="30.353" y2="5.715" width="0.8128" layer="1"/>
-<wire x1="30.353" y1="5.715" x2="32.385" y2="4.225" width="0.8128" layer="1"/>
+<wire x1="21.59" y1="4.225" x2="23.876" y2="5.08" width="0.8128" layer="1"/>
+<wire x1="23.876" y1="5.08" x2="30.607" y2="5.08" width="0.8128" layer="1"/>
+<wire x1="30.607" y1="5.08" x2="32.385" y2="4.225" width="0.8128" layer="1"/>
 <wire x1="32.385" y1="4.225" x2="33.701" y2="4.225" width="0.8128" layer="1"/>
 <wire x1="32.451" y1="2.475" x2="32.385" y2="2.475" width="0.8128" layer="1"/>
@@
 <wire x1="44.323" y1="15.748" x2="41.5036" y2="14.224" width="0.8128" layer="1"/>
 <wire x1="33.701" y1="10.225" x2="33.763" y2="10.287" width="0.8128" layer="1"/>
-<wire x1="33.763" y1="10.287" x2="41.783" y2="10.287" width="0.8128" layer="1"/>
-<wire x1="41.783" y1="10.287" x2="42.291" y2="10.287" width="0.8128" layer="1"/>
-<wire x1="42.291" y1="10.287" x2="44.323" y2="8.255" width="0.8128" layer="1"/>
+<wire x1="33.763" y1="10.287" x2="41.529" y2="10.287" width="0.8128" layer="1"/>
+<wire x1="41.529" y1="10.287" x2="41.656" y2="10.287" width="0.8128" layer="1"/>
+<wire x1="41.656" y1="10.287" x2="44.323" y2="8.255" width="0.8128" layer="1"/>
 <wire x1="41.5036" y1="14.1478" x2="41.5036" y2="10.5664" width="0.8128" layer="1"/>
-<wire x1="41.5036" y1="10.5664" x2="41.783" y2="10.287" width="0.8128" layer="1"/>
+<wire x1="41.5036" y1="10.5664" x2="41.529" y2="10.287" width="0.8128" layer="1"/>
 </signal>
 <signal name="KEY">
